Commit message: fixed urdfs

File: urdf/calibration/link5.xacro (robot description, xacro)
@@ -2,5 +2,5 @@
 <robot name="calibration_skin" xmlns:xacro="http://ros.org/wiki/xacro">
   <!-- Include the link5 skin macro -->
-  <xacro:include filename="$(find gentact_ros_tools)/urdf/skin/link5_fancy.xacro" />
+  <xacro:include filename="$(find gentact_descriptions)/urdf/skin/link5_fancy.xacro" />
   <!-- Create a base link for the calibration skin -->
   <link name="calibration_base" />

File: urdf/end_effectors/large_plate_ee.xacro (robot description, xacro)
@@ -2,6 +2,6 @@
 <robot xmlns:xacro="http://ros.org/wiki/xacro">
   <xacro:macro name="ee_macro" params="parent">
-    <xacro:include filename="$(find gentact_ros_tools)/urdf/end_effectors/ee_base.xacro" />
-    <xacro:property name="mesh_file" value="package://gentact_ros_tools/meshes/end_effectors/large_plate_ee.stl" />
+    <xacro:include filename="$(find gentact_descriptions)/urdf/end_effectors/ee_base.xacro" />
+    <xacro:property name="mesh_file" value="package://gentact_descriptions/meshes/end_effectors/large_plate_ee.stl" />
     <!-- Instantiate dermis once -->
     <xacro:ee_base_macro

File: urdf/end_effectors/sphere_ee.xacro (robot description, xacro)
@@ -2,6 +2,6 @@
 <robot xmlns:xacro="http://ros.org/wiki/xacro">
   <xacro:macro name="ee_macro" params="parent">
-    <xacro:include filename="$(find gentact_ros_tools)/urdf/end_effectors/ee_base.xacro" />
-    <xacro:property name="mesh_file" value="package://gentact_ros_tools/meshes/end_effectors/sphere_tip3.stl" />
+    <xacro:include filename="$(find gentact_descriptions)/urdf/end_effectors/ee_base.xacro" />
+    <xacro:property name="mesh_file" value="package://gentact_descriptions/meshes/end_effectors/sphere_tip3.stl" />
     <!-- Instantiate dermis once -->
     <xacro:ee_base_macro

File: urdf/skin/link1_fancy.xacro (robot description, xacro)
@@ -5,5 +5,5 @@
     <!-- Properties -->
     <xacro:property name="use_mesh_file" value="true" />
-    <xacro:property name="mesh_file" value="package://gentact_ros_tools/meshes/skin/self-cap/link1_fancy.stl" />
+    <xacro:property name="mesh_file" value="package://gentact_descriptions/meshes/skin/self-cap/link1_fancy.stl" />
     <xacro:property name="mass" value="0.3" /> <!-- [kg] -->
     <xacro:property name="body_width" value="0.3" /> <!-- [m] -->
@@ -12,5 +12,5 @@
     <xacro:property name="sensor_radius" value="0.0" /> <!-- [m] -->
     <!-- Included URDF Files -->
-    <xacro:include filename="$(find gentact_ros_tools)/urdf/skin/self-cap-base.xacro" />
+    <xacro:include filename="$(find gentact_descriptions)/urdf/skin/self-cap-base.xacro" />
     <!-- Instantiate dermis once -->
     <xacro:dermis_base_macro

File: urdf/skin/link2_fancy.xacro (robot description, xacro)
@@ -5,5 +5,5 @@
     <!-- Properties -->
     <xacro:property name="use_mesh_file" value="true" />
-    <xacro:property name="mesh_file" value="package://gentact_ros_tools/meshes/skin/self-cap/link2_fancy.stl" />
+    <xacro:property name="mesh_file" value="package://gentact_descriptions/meshes/skin/self-cap/link2_fancy.stl" />
     <xacro:property name="mass" value="0.3" /> <!-- [kg] -->
     <xacro:property name="body_width" value="0.3" /> <!-- [m] -->
@@ -12,5 +12,5 @@
     <xacro:property name="sensor_radius" value="0.0" /> <!-- [m] -->
     <!-- Included URDF Files -->
-    <xacro:include filename="$(find gentact_ros_tools)/urdf/skin/self-cap-base.xacro" />
+    <xacro:include filename="$(find gentact_descriptions)/urdf/skin/self-cap-base.xacro" />
     <!-- Instantiate dermis once -->
     <xacro:dermis_base_macro

File: urdf/skin/link3_fancy.xacro (robot description, xacro)
@@ -5,5 +5,5 @@
     <!-- Properties -->
     <xacro:property name="use_mesh_file" value="true" />
-    <xacro:property name="mesh_file" value="package://gentact_ros_tools/meshes/skin/self-cap/link3_fancy.stl" />
+    <xacro:property name="mesh_file" value="package://gentact_descriptions/meshes/skin/self-cap/link3_fancy.stl" />
     <xacro:property name="mass" value="0.3" /> <!-- [kg] -->
     <xacro:property name="body_width" value="0.3" /> <!-- [m] -->
@@ -12,5 +12,5 @@
     <xacro:property name="sensor_radius" value="0.0" /> <!-- [m] -->
     <!-- Included URDF Files -->
-    <xacro:include filename="$(find gentact_ros_tools)/urdf/skin/self-cap-base.xacro" />
+    <xacro:include filename="$(find gentact_descriptions)/urdf/skin/self-cap-base.xacro" />
     <!-- Instantiate dermis once -->
     <xacro:dermis_base_macro

File: urdf/skin/link4_fancy.xacro (robot description, xacro)
@@ -5,5 +5,5 @@
     <!-- Properties -->
     <xacro:property name="use_mesh_file" value="true" />
-    <xacro:property name="mesh_file" value="package://gentact_ros_tools/meshes/skin/self-cap/link4_fancy.stl" />
+    <xacro:property name="mesh_file" value="package://gentact_descriptions/meshes/skin/self-cap/link4_fancy.stl" />
     <xacro:property name="mass" value="0.3" /> <!-- [kg] -->
     <xacro:property name="body_width" value="0.3" /> <!-- [m] -->
@@ -12,5 +12,5 @@
     <xacro:property name="sensor_radius" value="0.0" /> <!-- [m] -->
     <!-- Included URDF Files -->
-    <xacro:include filename="$(find gentact_ros_tools)/urdf/skin/self-cap-base.xacro" />
+    <xacro:include filename="$(find gentact_descriptions)/urdf/skin/self-cap-base.xacro" />
     <!-- Instantiate dermis once -->
     <xacro:dermis_base_macro

File: urdf/skin/link5_fancy.xacro (robot description, xacro)
@@ -5,5 +5,5 @@
     <!-- Properties -->
     <xacro:property name="use_mesh_file" value="true" />
-    <xacro:property name="mesh_file" value="package://gentact_ros_tools/meshes/skin/self-cap/link5_fancy.stl" />
+    <xacro:property name="mesh_file" value="package://gentact_descriptions/meshes/skin/self-cap/link5_fancy.stl" />
     <xacro:property name="mass" value="0.3" /> <!-- [kg] -->
     <xacro:property name="body_width" value="0.3" /> <!-- [m] -->
@@ -12,5 +12,5 @@
     <xacro:property name="sensor_radius" value="0.0" /> <!-- [m] -->
     <!-- Included URDF Files -->
-    <xacro:include filename="$(find gentact_ros_tools)/urdf/skin/self-cap-base.xacro" />
+    <xacro:include filename="$(find gentact_descriptions)/urdf/skin/self-cap-base.xacro" />
     <!-- Instantiate dermis once -->
     <xacro:dermis_base_macro

File: urdf/skin/link5_spad.xacro (robot description, xacro)
@@ -5,5 +5,5 @@
     <!-- Properties -->
     <xacro:property name="use_mesh_file" value="true" />
-    <xacro:property name="mesh_file" value="package://gentact_ros_tools/meshes/skin/spad/link5_spad.stl" />
+    <xacro:property name="mesh_file" value="package://gentact_descriptions/meshes/skin/spad/link5_spad.stl" />
     <xacro:property name="mass" value="0.3" /> <!-- [kg] -->
     <xacro:property name="body_width" value="0.3" /> <!-- [m] -->
@@ -12,5 +12,5 @@
     <xacro:property name="sensor_radius" value="0.005" /> <!-- [m] -->
     <!-- Included URDF Files -->
-    <xacro:include filename="$(find gentact_ros_tools)/urdf/skin/self-cap-base.xacro" />
+    <xacro:include filename="$(find gentact_descriptions)/urdf/skin/self-cap-base.xacro" />
     <!-- Instantiate dermis once -->
     <xacro:dermis_base_macro

File: urdf/skin/link6_big.xacro (robot description, xacro)
@@ -5,5 +5,5 @@
     <!-- Properties -->
     <xacro:property name="use_mesh_file" value="true" />
-    <xacro:property name="mesh_file" value="package://gentact_ros_tools/meshes/skin/self-cap/link6_big.stl" />
+    <xacro:property name="mesh_file" value="package://gentact_descriptions/meshes/skin/self-cap/link6_big.stl" />
     <xacro:property name="mass" value="0.3" /> <!-- [kg] -->
     <xacro:property name="body_width" value="0.3" /> <!-- [m] -->
@@ -12,5 +12,5 @@
     <xacro:property name="sensor_radius" value="0.0" /> <!-- [m] -->
     <!-- Included URDF Files -->
-    <xacro:include filename="$(find gentact_ros_tools)/urdf/skin/self-cap-base.xacro" />
+    <xacro:include filename="$(find gentact_descriptions)/urdf/skin/self-cap-base.xacro" />
     <!-- Instantiate dermis once -->
     <xacro:dermis_base_macro

File: urdf/skin/link6_fancy.xacro (robot description, xacro)
@@ -5,5 +5,5 @@
     <!-- Properties -->
     <xacro:property name="use_mesh_file" value="true" />
-    <xacro:property name="mesh_file" value="package://gentact_ros_tools/meshes/skin/self-cap/link6_fancy.stl" />
+    <xacro:property name="mesh_file" value="package://gentact_descriptions/meshes/skin/self-cap/link6_fancy.stl" />
     <xacro:property name="mass" value="0.3" /> <!-- [kg] -->
     <xacro:property name="body_width" value="0.3" /> <!-- [m] -->
@@ -12,5 +12,5 @@
     <xacro:property name="sensor_radius" value="0.0" /> <!-- [m] -->
     <!-- Included URDF Files -->
-    <xacro:include filename="$(find gentact_ros_tools)/urdf/skin/self-cap-base.xacro" />
+    <xacro:include filename="$(find gentact_descriptions)/urdf/skin/self-cap-base.xacro" />
     <!-- Instantiate dermis once -->
     <xacro:dermis_base_macro
