Commit message: testing skin on h1-2

File: robots/h1-2/h1_2_handless.urdf.xacro (robot description, xacro)
@@ -1,5 +1,22 @@
-<robot name="h1_2">
+<?xml version="1.0"?>
+<robot xmlns:xacro="http://www.ros.org/wiki/xacro" name="h1_2">
+  <!-- Properties -->
+  <xacro:property name="mesh_dir" value="meshes" />
+  <!-- Material colors -->
+  <xacro:property name="material_grey" value="0.1 0.1 0.1 1" />
+  <xacro:property name="material_white" value="1 1 1 1" />
+  <!-- Material macro -->
+  <xacro:macro name="material_grey">
+    <material>
+      <color rgba="${material_grey}"/>
+    </material>
+  </xacro:macro>
+  <xacro:macro name="material_white">
+    <material>
+      <color rgba="${material_white}"/>
+    </material>
+  </xacro:macro>
   <mujoco>
-    <compiler meshdir="meshes" discardvisual="false"/>
+    <compiler meshdir="${mesh_dir}" discardvisual="false"/>
   </mujoco>
   <!-- [CAUTION] uncomment when convert to mujoco -->
@@ -18,14 +35,12 @@
       <origin xyz="0 0 0" rpy="0 0 0"/>
       <geometry>
-        <mesh filename="meshes/pelvis.STL"/>
-      </geometry>
-      <material>
-        <color rgba="0.1 0.1 0.1 1"/>
-      </material>
-    </visual>
-    <collision>
-      <origin xyz="0 0 0" rpy="0 0 0"/>
-      <geometry>
-        <mesh filename="meshes/pelvis.STL"/>
+        <mesh filename="${mesh_dir}/pelvis.STL"/>
+      </geometry>
+      <xacro:material_grey />
+    </visual>
+    <collision>
+      <origin xyz="0 0 0" rpy="0 0 0"/>
+      <geometry>
+        <mesh filename="${mesh_dir}/pelvis.STL"/>
       </geometry>
     </collision>
@@ -41,9 +56,7 @@
       <origin xyz="0 0 0" rpy="0 0 0"/>
       <geometry>
-        <mesh filename="meshes/left_hip_yaw_link.STL"/>
-      </geometry>
-      <material>
-        <color rgba="0.1 0.1 0.1 1"/>
-      </material>
+        <mesh filename="${mesh_dir}/left_hip_yaw_link.STL"/>
+      </geometry>
+      <xacro:material_grey />
     </visual>
   </link>
@@ -64,14 +77,12 @@
       <origin xyz="0 0 0" rpy="0 0 0"/>
       <geometry>
-        <mesh filename="meshes/left_hip_pitch_link.STL"/>
-      </geometry>
-      <material>
-        <color rgba="0.1 0.1 0.1 1"/>
-      </material>
-    </visual>
-    <collision>
-      <origin xyz="0 0 0" rpy="0 0 0"/>
-      <geometry>
-        <mesh filename="meshes/left_hip_pitch_link.STL"/>
+        <mesh filename="${mesh_dir}/left_hip_pitch_link.STL"/>
+      </geometry>
+      <xacro:material_grey />
+    </visual>
+    <collision>
+      <origin xyz="0 0 0" rpy="0 0 0"/>
+      <geometry>
+        <mesh filename="${mesh_dir}/left_hip_pitch_link.STL"/>
       </geometry>
     </collision>
@@ -93,14 +104,12 @@
       <origin xyz="0 0 0" rpy="0 0 0"/>
       <geometry>
-        <mesh filename="meshes/left_hip_roll_link.STL"/>
-      </geometry>
-      <material>
-        <color rgba="0.1 0.1 0.1 1"/>
-      </material>
-    </visual>
-    <collision>
-      <origin xyz="0 0 0" rpy="0 0 0"/>
-      <geometry>
-        <mesh filename="meshes/left_hip_roll_link.STL"/>
+        <mesh filename="${mesh_dir}/left_hip_roll_link.STL"/>
+      </geometry>
+      <xacro:material_grey />
+    </visual>
+    <collision>
+      <origin xyz="0 0 0" rpy="0 0 0"/>
+      <geometry>
+        <mesh filename="${mesh_dir}/left_hip_roll_link.STL"/>
       </geometry>
     </collision>
@@ -122,9 +131,7 @@
       <origin xyz="0 0 0" rpy="0 0 0"/>
       <geometry>
-        <mesh filename="meshes/left_knee_link.STL"/>
-      </geometry>
-      <material>
-        <color rgba="0.1 0.1 0.1 1"/>
-      </material>
+        <mesh filename="${mesh_dir}/left_knee_link.STL"/>
+      </geometry>
+      <xacro:material_grey />
     </visual>
     <collision>
@@ -151,9 +158,7 @@
       <origin xyz="0 0 0" rpy="0 0 0"/>
       <geometry>
-        <mesh filename="meshes/left_ankle_pitch_link.STL"/>
-      </geometry>
-      <material>
-        <color rgba="0.1 0.1 0.1 1"/>
-      </material>
+        <mesh filename="${mesh_dir}/left_ankle_pitch_link.STL"/>
+      </geometry>
+      <xacro:material_grey />
     </visual>
   </link>
@@ -174,14 +179,12 @@
       <origin xyz="0 0 0" rpy="0 0 0"/>
       <geometry>
-        <mesh filename="meshes/left_ankle_roll_link.STL"/>
-      </geometry>
-      <material>
-        <color rgba="0.1 0.1 0.1 1"/>
-      </material>
-    </visual>
-    <collision>
-      <origin xyz="0 0 0" rpy="0 0 0"/>
-      <geometry>
-        <mesh filename="meshes/left_ankle_roll_link.STL"/>
+        <mesh filename="${mesh_dir}/left_ankle_roll_link.STL"/>
+      </geometry>
+      <xacro:material_grey />
+    </visual>
+    <collision>
+      <origin xyz="0 0 0" rpy="0 0 0"/>
+      <geometry>
+        <mesh filename="${mesh_dir}/left_ankle_roll_link.STL"/>
       </geometry>
     </collision>
@@ -204,9 +207,7 @@
       <origin xyz="0 0 0" rpy="0 0 0"/>
       <geometry>
-        <mesh filename="meshes/right_hip_yaw_link.STL"/>
-      </geometry>
-      <material>
-        <color rgba="0.1 0.1 0.1 1"/>
-      </material>
+        <mesh filename="${mesh_dir}/right_hip_yaw_link.STL"/>
+      </geometry>
+      <xacro:material_grey />
     </visual>
   </link>
@@ -227,14 +228,12 @@
       <origin xyz="0 0 0" rpy="0 0 0"/>
       <geometry>
-        <mesh filename="meshes/right_hip_pitch_link.STL"/>
-      </geometry>
-      <material>
-        <color rgba="0.1 0.1 0.1 1"/>
-      </material>
-    </visual>
-    <collision>
-      <origin xyz="0 0 0" rpy="0 0 0"/>
-      <geometry>
-        <mesh filename="meshes/right_hip_pitch_link.STL"/>
+        <mesh filename="${mesh_dir}/right_hip_pitch_link.STL"/>
+      </geometry>
+      <xacro:material_grey />
+    </visual>
+    <collision>
+      <origin xyz="0 0 0" rpy="0 0 0"/>
+      <geometry>
+        <mesh filename="${mesh_dir}/right_hip_pitch_link.STL"/>
       </geometry>
     </collision>
@@ -256,14 +255,12 @@
       <origin xyz="0 0 0" rpy="0 0 0"/>
       <geometry>
-        <mesh filename="meshes/right_hip_roll_link.STL"/>
-      </geometry>
-      <material>
-        <color rgba="0.1 0.1 0.1 1"/>
-      </material>
-    </visual>
-    <collision>
-      <origin xyz="0 0 0" rpy="0 0 0"/>
-      <geometry>
-        <mesh filename="meshes/right_hip_roll_link.STL"/>
+        <mesh filename="${mesh_dir}/right_hip_roll_link.STL"/>
+      </geometry>
+      <xacro:material_grey />
+    </visual>
+    <collision>
+      <origin xyz="0 0 0" rpy="0 0 0"/>
+      <geometry>
+        <mesh filename="${mesh_dir}/right_hip_roll_link.STL"/>
       </geometry>
     </collision>
@@ -285,9 +282,7 @@
       <origin xyz="0 0 0" rpy="0 0 0"/>
       <geometry>
-        <mesh filename="meshes/right_knee_link.STL"/>
-      </geometry>
-      <material>
-        <color rgba="0.1 0.1 0.1 1"/>
-      </material>
+        <mesh filename="${mesh_dir}/right_knee_link.STL"/>
+      </geometry>
+      <xacro:material_grey />
     </visual>
     <collision>
@@ -314,9 +309,7 @@
       <origin xyz="0 0 0" rpy="0 0 0"/>
       <geometry>
-        <mesh filename="meshes/right_ankle_pitch_link.STL"/>
-      </geometry>
-      <material>
-        <color rgba="0.1 0.1 0.1 1"/>
-      </material>
+        <mesh filename="${mesh_dir}/right_ankle_pitch_link.STL"/>
+      </geometry>
+      <xacro:material_grey />
     </visual>
   </link>
@@ -337,14 +330,12 @@
       <origin xyz="0 0 0" rpy="0 0 0"/>
       <geometry>
-        <mesh filename="meshes/right_ankle_roll_link.STL"/>
-      </geometry>
-      <material>
-        <color rgba="0.1 0.1 0.1 1"/>
-      </material>
-    </visual>
-    <collision>
-      <origin xyz="0 0 0" rpy="0 0 0"/>
-      <geometry>
-        <mesh filename="meshes/right_ankle_roll_link.STL"/>
+        <mesh filename="${mesh_dir}/right_ankle_roll_link.STL"/>
+      </geometry>
+      <xacro:material_grey />
+    </visual>
+    <collision>
+      <origin xyz="0 0 0" rpy="0 0 0"/>
+      <geometry>
+        <mesh filename="${mesh_dir}/right_ankle_roll_link.STL"/>
       </geometry>
     </collision>
@@ -367,14 +358,12 @@
       <origin xyz="0 0 0" rpy="0 0 0"/>
       <geometry>
-        <mesh filename="meshes/torso_link.STL"/>
-      </geometry>
-      <material>
-        <color rgba="0.1 0.1 0.1 1"/>
-      </material>
-    </visual>
-    <collision>
-      <origin xyz="0 0 0" rpy="0 0 0"/>
-      <geometry>
-        <mesh filename="meshes/torso_link.STL"/>
+        <mesh filename="${mesh_dir}/torso_link.STL"/>
+      </geometry>
+      <xacro:material_grey />
+    </visual>
+    <collision>
+      <origin xyz="0 0 0" rpy="0 0 0"/>
+      <geometry>
+        <mesh filename="${mesh_dir}/torso_link.STL"/>
       </geometry>
     </collision>
@@ -397,14 +386,12 @@
       <origin xyz="0 0 0" rpy="0 0 0"/>
       <geometry>
-        <mesh filename="meshes/left_shoulder_pitch_link.STL"/>
-      </geometry>
-      <material>
-        <color rgba="0.1 0.1 0.1 1"/>
-      </material>
-    </visual>
-    <collision>
-      <origin xyz="0 0 0" rpy="0 0 0"/>
-      <geometry>
-        <mesh filename="meshes/left_shoulder_pitch_link.STL"/>
+        <mesh filename="${mesh_dir}/left_shoulder_pitch_link.STL"/>
+      </geometry>
+      <xacro:material_grey />
+    </visual>
+    <collision>
+      <origin xyz="0 0 0" rpy="0 0 0"/>
+      <geometry>
+        <mesh filename="${mesh_dir}/left_shoulder_pitch_link.STL"/>
       </geometry>
     </collision>
@@ -426,14 +413,12 @@
       <origin xyz="0 0 0" rpy="0 0 0"/>
       <geometry>
-        <mesh filename="meshes/left_shoulder_roll_link.STL"/>
-      </geometry>
-      <material>
-        <color rgba="0.1 0.1 0.1 1"/>
-      </material>
-    </visual>
-    <collision>
-      <origin xyz="0 0 0" rpy="0 0 0"/>
-      <geometry>
-        <mesh filename="meshes/left_shoulder_roll_link.STL"/>
+        <mesh filename="${mesh_dir}/left_shoulder_roll_link.STL"/>
+      </geometry>
+      <xacro:material_grey />
+    </visual>
+    <collision>
+      <origin xyz="0 0 0" rpy="0 0 0"/>
+      <geometry>
+        <mesh filename="${mesh_dir}/left_shoulder_roll_link.STL"/>
       </geometry>
     </collision>
@@ -455,14 +440,12 @@
       <origin xyz="0 0 0" rpy="0 0 0"/>
       <geometry>
-        <mesh filename="meshes/left_shoulder_yaw_link.STL"/>
-      </geometry>
-      <material>
-        <color rgba="0.1 0.1 0.1 1"/>
-      </material>
-    </visual>
-    <collision>
-      <origin xyz="0 0 0" rpy="0 0 0"/>
-      <geometry>
-        <mesh filename="meshes/left_shoulder_yaw_link.STL"/>
+        <mesh filename="${mesh_dir}/left_shoulder_yaw_link.STL"/>
+      </geometry>
+      <xacro:material_grey />
+    </visual>
+    <collision>
+      <origin xyz="0 0 0" rpy="0 0 0"/>
+      <geometry>
+        <mesh filename="${mesh_dir}/left_shoulder_yaw_link.STL"/>
       </geometry>
     </collision>
@@ -484,14 +467,12 @@
       <origin xyz="0 0 0" rpy="0 0 0"/>
       <geometry>
-        <mesh filename="meshes/left_elbow_link.STL"/>
-      </geometry>
-      <material>
-        <color rgba="0.1 0.1 0.1 1"/>
-      </material>
-    </visual>
-    <collision>
-      <origin xyz="0 0 0" rpy="0 0 0"/>
-      <geometry>
-        <mesh filename="meshes/left_elbow_link.STL"/>
+        <mesh filename="${mesh_dir}/left_elbow_link.STL"/>
+      </geometry>
+      <xacro:material_grey />
+    </visual>
+    <collision>
+      <origin xyz="0 0 0" rpy="0 0 0"/>
+      <geometry>
+        <mesh filename="${mesh_dir}/left_elbow_link.STL"/>
       </geometry>
     </collision>
@@ -513,13 +494,11 @@
       <origin xyz="0 0 0" rpy="0 0 0"/>
       <geometry>
-        <mesh filename="meshes/left_wrist_roll_link.STL"/>
-      </geometry>
-      <material>
-        <color rgba="0.1 0.1 0.1 1"/>
-      </material>
-    </visual>
-    <collision>
-      <geometry>
-        <mesh filename="meshes/left_wrist_roll_link.STL"/>
+        <mesh filename="${mesh_dir}/left_wrist_roll_link.STL"/>
+      </geometry>
+      <xacro:material_grey />
+    </visual>
+    <collision>
+      <geometry>
+        <mesh filename="${mesh_dir}/left_wrist_roll_link.STL"/>
       </geometry>
     </collision>
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
File: robots/h1-2/h1_2_handless_skintest.urdf (robot description, URDF)
Before this commit: robot h1_2, 32 links, 31 joints
Links:
- added link right_shoulder_roll_sensor_0; collision sphere radius=0.0; visual sphere radius=0.0
- added link right_shoulder_roll_sensor_1; collision sphere radius=0.0; visual sphere radius=0.0
- added link right_shoulder_roll_sensor_2; collision sphere radius=0.0; visual sphere radius=0.0
- added link right_shoulder_roll_sensor_3; collision sphere radius=0.0; visual sphere radius=0.0
- added link right_shoulder_roll_sensor_4; collision sphere radius=0.0; visual sphere radius=0.0
- added link right_shoulder_roll_sensor_5; collision sphere radius=0.0; visual sphere radius=0.0
- added link right_shoulder_roll_sensor_6; collision sphere radius=0.0; visual sphere radius=0.0
- added link right_shoulder_roll_sensor_7; collision sphere radius=0.0; visual sphere radius=0.0
- added link right_shoulder_roll_skin; visual mesh filename= scale=1 1 1
Joints:
- added joint right_shoulder_roll_base_joint: type fixed, parent right_shoulder_roll_link, child right_shoulder_roll_skin, origin xyz=0 0 0 rpy=1.5707 0 0
- added joint right_shoulder_roll_sensor_0_joint: type fixed, parent right_shoulder_roll_skin, child right_shoulder_roll_sensor_0, origin xyz=0.02020913176238537 -0.010433539748191833 -0.1203891709446907 rpy=1.6110156774520874 -1.3015655042636354e-07 1.3825271129608154, axis 0.9815351963043213 -0.18700765073299408 -0.04020834341645241
- added joint right_shoulder_roll_sensor_1_joint: type fixed, parent right_shoulder_roll_skin, child right_shoulder_roll_sensor_1, origin xyz=0.02196035161614418 0.003525834996253252 0.006447893101722002 rpy=1.547227382659912 1.2260383641660155e-07 1.5840967893600464, axis 0.9996338486671448 0.013296284712851048 0.023566756397485733
- added joint right_shoulder_roll_sensor_2_joint: type fixed, parent right_shoulder_roll_skin, child right_shoulder_roll_sensor_2, origin xyz=0.021171631291508675 -0.013482555747032166 -0.03812651336193085 rpy=1.6198302507400513 3.5244884344365346e-08 1.4298112392425537, axis 0.9888880252838135 -0.14034967124462128 -0.04901430755853653
- added joint right_shoulder_roll_sensor_3_joint: type fixed, parent right_shoulder_roll_skin, child right_shoulder_roll_sensor_3, origin xyz=0.019492628052830696 -0.013848518952727318 -0.07953478395938873 rpy=1.5781761407852173 -1.408326113505609e-07 1.3229039907455444, axis 0.9694053530693054 -0.24535463750362396 -0.007379625923931599
- added joint right_shoulder_roll_sensor_4_joint: type fixed, parent right_shoulder_roll_skin, child right_shoulder_roll_sensor_4, origin xyz=0.011047429405152798 0.03214484453201294 -0.08381814509630203 rpy=1.5731147527694702 -3.6292128413606406e-08 2.1917271614074707, axis 0.8133350610733032 0.5817909836769104 -0.002318537561222911
- added joint right_shoulder_roll_sensor_5_joint: type fixed, parent right_shoulder_roll_skin, child right_shoulder_roll_sensor_5, origin xyz=-0.0885578915476799 0.008191447705030441 -0.12311510741710663 rpy=1.6344798803329468 4.719517221474234e-08 -1.7226282358169556, axis -0.9864919185638428 0.15094248950481415 -0.06364033371210098
- added joint right_shoulder_roll_sensor_6_joint: type fixed, parent right_shoulder_roll_skin, child right_shoulder_roll_sensor_6, origin xyz=-0.043252378702163696 -0.05412545055150986 -0.12589296698570251 rpy=1.6463441848754883 -1.1537085065072006e-08 -0.16923603415489197, axis -0.1679488718509674 -0.9829021096229553 -0.07547598332166672
- added joint right_shoulder_roll_sensor_7_joint: type fixed, parent right_shoulder_roll_skin, child right_shoulder_roll_sensor_7, origin xyz=-0.010976525023579597 0.05005709081888199 -0.12077049911022186 rpy=1.6160632371902466 -1.495763335412903e-08 2.7067909240722656, axis 0.4207991361618042 0.9060245156288147 -0.04525141045451164
