Commit message: testing skin unit on h1-2

File: robots/h1-2/h1_2_handless_skintest.urdf (robot description, URDF)
Before this commit: robot h1_2, 41 links, 40 joints
Joints:
- joint right_shoulder_roll_base_joint: origin xyz=0 0 0 rpy=1.5707 0 0 -> xyz=0 0 0 rpy=0 0 0

File: robots/h1-2/skin/right_shoulder_roll_skin.xacro (robot description, xacro)
@@ -22,5 +22,5 @@
     use_mesh_file="${use_mesh_file}"
     mesh_file="${mesh_file}">
-    <origin xyz="0 0 0" rpy="1.5707 0 0" />
+    <origin xyz="0 0 0" rpy="0 0 0" />
     </xacro:dermis_base_macro>
     <xacro:self_cap_sensor
