Commit message: Link6 working for trybrid

File: robots/common/trimodal_unit_base.xacro (robot description, xacro)
@@ -49,3 +49,23 @@
     </link>
   </xacro:macro>
+  <!-- ToF Sensor -->
+  <xacro:macro name="tof_sensor"
+    params="robot_namespace parent sensor_number *origin">
+    <joint name="${robot_namespace}_tof_sensor_${sensor_number}_joint" type="fixed">
+      <xacro:insert_block name="origin" />
+      <parent link="${parent}" />
+      <child link="${robot_namespace}_tof_sensor_${sensor_number}" />
+    </joint>
+    <link name="${robot_namespace}_tof_sensor_${sensor_number}" />
+  </xacro:macro>
+  <!-- Magnetic Sensor -->
+  <xacro:macro name="mag_sensor"
+    params="robot_namespace parent sensor_number *origin">
+    <joint name="${robot_namespace}_mag_sensor_${sensor_number}_joint" type="fixed">
+      <xacro:insert_block name="origin" />
+      <parent link="${parent}" />
+      <child link="${robot_namespace}_mag_sensor_${sensor_number}" />
+    </joint>
+    <link name="${robot_namespace}_mag_sensor_${sensor_number}" />
+  </xacro:macro>
 </robot>

File: robots/skin/trimodal/link6_base.xacro (robot description, xacro)
@@ -34,5 +34,5 @@
       normal_y="-0.771"
       normal_z="-0.155">
-      <origin xyz="-0.0631 -0.0491 -0.0215" rpy="1.726 0.000 -0.676" />
+      <origin xyz="0.125 0.007 -0.044" rpy="-2.235 -0.896 -0.784" />
     </xacro:self_cap_sensor>
     <xacro:self_cap_sensor
@@ -45,5 +45,5 @@
       normal_y="-0.709"
       normal_z="0.702">
-      <origin xyz="-0.0353 -0.0490 0.0221" rpy="0.793 0.000 -0.103" />
+      <origin xyz="0.099 0.041 -0.028" rpy="-1.643 -0.025 -0.337" />
     </xacro:self_cap_sensor>
     <xacro:self_cap_sensor
@@ -56,6 +56,38 @@
       normal_y="-0.117"
       normal_z="0.014">
-      <origin xyz="0.0913 -0.0053 -0.0027" rpy="1.557 -0.000 1.454" />
+      <origin xyz="0.110 -0.036 -0.032" rpy="1.863 -0.257 0.703" />
     </xacro:self_cap_sensor>
+    <!-- Instantiate self ToF sensor -->
+    <xacro:tof_sensor
+      robot_namespace="${namespace}"
+      parent="${namespace}_skin"
+      sensor_number="0">
+      <origin xyz="0.105 0.007 -0.077" rpy="-2.837 -0.800 -0.222" />
+    </xacro:tof_sensor>
+        <xacro:tof_sensor
+      robot_namespace="${namespace}"
+      parent="${namespace}_skin"
+      sensor_number="1">
+      <origin xyz="0.081 0.041 -0.058" rpy="-1.861 -0.033 -0.110" />
+    </xacro:tof_sensor>
+        <xacro:tof_sensor
+      robot_namespace="${namespace}"
+      parent="${namespace}_skin"
+      sensor_number="2">
+      <origin xyz="0.089 -0.037 -0.063" rpy="2.023 -0.158 0.313" />
+    </xacro:tof_sensor>
+    <!-- Instantiate magnetic sensor -->
+    <xacro:mag_sensor
+      robot_namespace="${namespace}"
+      parent="${namespace}_skin"
+      sensor_number="0">
+      <origin xyz="0.118 -0.023 -0.045" rpy="1.877 -0.320 0.783" />
+    </xacro:mag_sensor>
+    <xacro:mag_sensor
+      robot_namespace="${namespace}"
+      parent="${namespace}_skin"
+      sensor_number="1">
+      <origin xyz="0.107 0.036 -0.039" rpy="-1.777 -0.095 -0.426" />
+    </xacro:mag_sensor>
   </xacro:macro>
 </robot>
